Commit message: Added camera

File: schunk_lwa4p_description/urdf/lwa4p.gazebo.xacro (robot description, xacro)
@@ -43,4 +43,50 @@
       <material value="Schunk/LightGrey" />
     </gazebo>
+	  <!-- camera_link -->
+  	<gazebo reference="camera_link">
+      <mu1>0.2</mu1>
+      <mu2>0.2</mu2>
+      <material value="Schunk/Black" />
+    </gazebo>
+	<!-- camera -->
+    <gazebo reference="camera_link">
+      <sensor type="camera" name="camera1">
+        <update_rate>30.0</update_rate>
+        <camera name="head">
+          <horizontal_fov>1.3962634</horizontal_fov>
+          <image>
+            <width>800</width>
+            <height>800</height>
+            <format>R8G8B8</format>
+          </image>
+          <clip>
+            <near>0.02</near>
+            <far>300</far>
+          </clip>
+          <noise>
+            <type>gaussian</type>
+           <!-- Noise is sampled independently per pixel on each frame.
+                That pixel's noise value is added to each of its color
+                channels, which at that point lie in the range [0,1]. -->
+            <mean>0.0</mean>
+            <stddev>0.007</stddev>
+          </noise>
+        </camera>
+        <plugin name="camera_controller" filename="libgazebo_ros_camera.so">
+          <alwaysOn>true</alwaysOn>
+          <updateRate>0.0</updateRate>
+          <cameraName>schunk_lwa4p/camera1</cameraName>
+          <imageTopicName>image_raw</imageTopicName>
+          <cameraInfoTopicName>camera_info</cameraInfoTopicName>
+          <frameName>camera_link_optical</frameName>
+          <hackBaseline>0.07</hackBaseline>
+          <distortionK1>0.0</distortionK1>
+          <distortionK2>0.0</distortionK2>
+          <distortionK3>0.0</distortionK3>
+          <distortionT1>0.0</distortionT1>
+          <distortionT2>0.0</distortionT2>
+        </plugin>
+      </sensor>
+    </gazebo>
   </xacro:macro>
 </robot>

File: schunk_lwa4p_description/urdf/lwa4p.urdf.xacro (robot description, xacro)
@@ -225,4 +225,45 @@
       </collision>
     </link>
+	<!-- joint between arm_6_link and camera -->
+	<joint name="camera_joint" type="fixed">
+      <axis xyz="0 0 0" />
+      <origin xyz="0 0 0.085" rpy="0 0 0"/>
+      <parent link="${name}_6_link"/>
+      <child link="camera_link"/>
+    </joint>
+	<xacro:property name="camera_box" value="0.05" /> <!-- Size of square 'camera' box -->
+	<!-- Camera -->
+    <link name="camera_link">
+	  <!-- <xacro:default_inertial/> -->
+      <collision>
+        <origin xyz="0 0 0" rpy="0 0 0"/>
+        <geometry>
+      <box size="${camera_box} ${camera_box/2} ${camera_box*3}"/>
+        </geometry>
+      </collision>
+      <visual>
+        <origin xyz="0 0 0" rpy="0 0 0"/>
+        <geometry>
+      <box size="${camera_box} ${camera_box/2} ${camera_box*3}"/>
+        </geometry>
+		<material name="Schunk/Black"/>
+      </visual>
+      <inertial>
+        <mass value="1e-5" />
+        <origin xyz="0 0 0" rpy="0 0 0"/>
+        <inertia ixx="1e-6" ixy="0" ixz="0" iyy="1e-6" iyz="0" izz="1e-6" />
+      </inertial>
+    </link>
+    <!-- generate an optical frame http://www.ros.org/reps/rep-0103.html#suffix-frames
+        so that ros and opencv can operate on the camera frame correctly -->
+    <joint name="camera_optical_joint" type="fixed">
+      <!-- these values have to be these values otherwise the gazebo camera image
+          won't be aligned properly with the frame it is supposedly originating from -->
+      <origin xyz="0 0 0" rpy="${-pi/2} 0 ${-pi/2}"/>
+      <parent link="camera_link"/>
+      <child link="camera_link_optical"/>
+    </joint>
+    <link name="camera_link_optical">
+    </link>
     <!-- extensions -->
     <xacro:schunk_lwa4p_gazebo name="${name}" />
