Commit message: Final version

File: schunk_lwa4p_description/calibration/calibration.urdf.xacro (robot description, xacro)
@@ -8,3 +8,5 @@
 	<property name="arm_5_ref" value="0" />
 	<property name="arm_6_ref" value="0" />
+    <!-- Size of square 'camera' box -->
+    <property name="camera_box" value="0.01" />
 </robot>

File: schunk_lwa4p_description/urdf/lwa4p.gazebo.xacro (robot description, xacro)
@@ -3,5 +3,5 @@
   <gazebo>
     <plugin name="gazebo_ros_control" filename="libgazebo_ros_control.so">
-      <robotNamespace>/lwa4p</robotNamespace>
+      <robotNamespace>/lwa4p_blue</robotNamespace>
       <robotSimType>gazebo_ros_control/DefaultRobotHWSim</robotSimType>
     </plugin>
@@ -54,5 +54,5 @@
         <update_rate>30.0</update_rate>
         <camera name="head">
-          <horizontal_fov>1.3962634</horizontal_fov>
+          <horizontal_fov>${M_PI/3}</horizontal_fov>
           <image>
             <width>800</width>
@@ -62,5 +62,5 @@
           <clip>
             <near>0.02</near>
-            <far>300</far>
+            <far>100</far>
           </clip>
           <noise>

File: schunk_lwa4p_description/urdf/lwa4p.urdf.xacro (robot description, xacro)
@@ -226,26 +226,25 @@
     </link>
 	<!-- joint between arm_6_link and camera -->
-	<joint name="camera_joint" type="fixed">
+    <joint name="camera_joint" type="fixed">
       <axis xyz="0 0 0" />
-      <origin xyz="0 0 0.085" rpy="0 0 0"/>
+      <origin xyz="0 0 0.09" rpy="0 ${-M_PI/2} ${M_PI}"/>
       <parent link="${name}_6_link"/>
       <child link="camera_link"/>
     </joint>
-	<xacro:property name="camera_box" value="0.05" /> <!-- Size of square 'camera' box -->
 	<!-- Camera -->
     <link name="camera_link">
-	  <!-- <xacro:default_inertial/> -->
-      <collision>
-        <origin xyz="0 0 0" rpy="0 0 0"/>
-        <geometry>
-      <box size="${camera_box} ${camera_box/2} ${camera_box*3}"/>
-        </geometry>
-      </collision>
-      <visual>
-        <origin xyz="0 0 0" rpy="0 0 0"/>
-        <geometry>
-      <box size="${camera_box} ${camera_box/2} ${camera_box*3}"/>
-        </geometry>
-		<material name="Schunk/Black"/>
+        <!-- <xacro:default_inertial/> -->
+      <collision>
+        <origin xyz="0 0 0" rpy="0 0 0"/>
+        <geometry>
+      <box size="${camera_box} ${camera_box*11} ${camera_box*5}"/>
+        </geometry>
+      </collision>
+      <visual>
+        <origin xyz="0 0 0" rpy="0 0 0"/>
+        <geometry>
+      <box size="${camera_box} ${camera_box*11} ${camera_box*5}"/>
+        </geometry>
+		<material name="Gazebo/Black"/>
       </visual>
       <inertial>
@@ -257,8 +256,8 @@
     <!-- generate an optical frame http://www.ros.org/reps/rep-0103.html#suffix-frames
         so that ros and opencv can operate on the camera frame correctly -->
-    <joint name="camera_optical_joint" type="fixed">
+     <joint name="camera_optical_joint" type="fixed">
       <!-- these values have to be these values otherwise the gazebo camera image
           won't be aligned properly with the frame it is supposedly originating from -->
-      <origin xyz="0 0 0" rpy="${-pi/2} 0 ${-pi/2}"/>
+    <origin xyz="0 0 0" rpy="0 0 0"/>
       <parent link="camera_link"/>
       <child link="camera_link_optical"/>

File: schunk_lwa4p_description/urdf/schunk_lwa4p.urdf.xacro (robot description, xacro)
@@ -1,3 +1,4 @@
 <?xml version="1.0"?>
+<!--
 <robot xmlns:sensor="http://playerstage.sourceforge.net/gazebo/xmlschema/#sensor"
        xmlns:controller="http://playerstage.sourceforge.net/gazebo/xmlschema/#controller"
@@ -5,4 +6,6 @@
        xmlns:xacro="http://playerstage.sourceforge.net/gazebo/xmlschema/#interface"
        name="lwa4p" >
+       -->
+<robot name="lwa4p" xmlns:xacro="http://www.ros.org/wiki/xacro" >
   	<!-- common stuff -->
  	<include filename="$(find cob_description)/urdf/common.xacro" />
